File: 1.kicad_pcb (KiCad board)
At the start: 2 copper layers, 71.1 x 43.2 mm, 29 parts, among them J1 Screw_Terminal_01x03, J2 Screw_Terminal_01x01, J3 Screw_Terminal_01x01, J4 Conn_01x03_Pin, J5 Screw_Terminal_01x01, J6 Screw_Terminal_01x01, J7 Conn_01x01_Pin, J8 Conn_01x04_Pin, J9 Conn_01x01_Pin, U1 LTC2990

Commit message: Fixes
Parts:
- Boost_IC1: footprint Boost LTC3426:SOT95P280X90-6N -> libs:SOT95P280X90-6N
- Buck_IC1: footprint BUck TPS62203DBVT:SOT95P280X145-5N -> libs:SOT95P280X145-5N
- C1, C4: footprint 10uF MLCC:CAPC2012X94N -> libs:CAPC2012X94N
- C2: footprint cap 22uF low esr and esl:C3216_Commercial -> libs:C3216_Commercial
- C3: footprint cap 4.7uf:C1210 -> libs:C1210
- D1: footprint Schottky DD with stock:DIOM5126X265N -> libs:DIOM5126X265N
- J1, J4: footprint TerminalBlock_Phoenix:TerminalBlock_Phoenix_MKDS-1,5-3_1x03_P5.00mm_Horizontal -> libs:TerminalBlock_Phoenix_MKDS-1,5-3_1x03_P5.00mm_Horizontal
- J2, J3, J5, J6: footprint Connector_Pin:Pin_D1.3mm_L11.0mm_LooseFit -> libs:Pin_D1.3mm_L11.0mm_LooseFit
- J7, J9: footprint Connector_PinHeader_2.54mm:PinHeader_1x01_P2.54mm_Vertical -> libs:PinHeader_1x01_P2.54mm_Vertical
- J8: footprint Connector_PinHeader_2.54mm:PinHeader_1x04_P2.54mm_Vertical -> libs:PinHeader_1x04_P2.54mm_Vertical
- JMP1: footprint Connector_PinHeader_2.54mm:PinHeader_1x02_P2.54mm_Vertical -> libs:PinHeader_1x02_P2.54mm_Vertical
- L1: footprint indc 2.2uH:IHLP2020CZER2R2M8A -> libs:IHLP2020CZER2R2M8A
- L2: footprint indc 10uH crct:SRN1060-100M -> libs:SRN1060-100M
- R1: footprint rst 95.3k:RESC2012X60N -> libs:RESC2012X60N
- R2: footprint rst 30.9k:RC0603FR-0730K9L -> libs:RC0603FR-0730K9L
- R3: footprint 1MEGA RST:RESC1608X55N -> libs:RESC1608X55N
- R5: footprint 50m RST:RESC3216X88N -> libs:RESC3216X88N
- TP1, TP3, TP5: footprint TestPoint:TestPoint_THTPad_1.5x1.5mm_Drill0.7mm -> libs:TestPoint_THTPad_1.5x1.5mm_Drill0.7mm
- TP8, TP9: footprint TestPoint:TestPoint_2Pads_Pitch2.54mm_Drill0.8mm -> libs:TestPoint_2Pads_Pitch2.54mm_Drill0.8mm
- U1: footprint MON & PROTECC:SOP50P490X110-10N -> libs:SOP50P490X110-10N
- moved J2 2.54 mm to (113.8, 71.1)
- moved J6 2.54 mm to (175.3, 71.1)
Other:
- board size 71.1 x 43.2 mm -> 68.6 x 40.6 mm
